Commit message: Tour guide robot updates: exhibit navigator, waypoint patrol, Pi/LLM integration, SLAM toolbox, navigation tuning

File: src/shbat_pkg/urdf/sahabat_robot.urdf.xacro (robot description, xacro)
@@ -1,5 +1,18 @@
 <?xml version = "1.0"?>
 <robot name="sahabat_robot" xmlns:xacro="http://www.ros.org/wiki/xacro">
-<!-- Parameters -->
+<!-- ================================================== -->
+<!-- Robot Parameters (edit these to match your robot)  -->
+<!-- ================================================== -->
+<!-- Wheel dimensions: 175mm diameter hoverboard wheels -->
+<xacro:property name="wheel_radius" value="0.0875" />   <!-- 175mm / 2 = 87.5mm -->
+<xacro:property name="wheel_width" value="0.057" />     <!-- Wheel width/thickness -->
+<xacro:property name="wheel_base" value="0.33" />       <!-- Distance between wheels (center to center) -->
+<!-- Caster wheel radius -->
+<xacro:property name="caster_radius" value="0.03" />
+<!-- Body dimensions -->
+<xacro:property name="body_length" value="0.3" />
+<xacro:property name="body_width" value="0.35" />
+<xacro:property name="body_height" value="0.22" />
+<!-- Camera arguments -->
 <xacro:arg name="camera_name" default="zed2i" />
 <xacro:arg name="camera_model" default="zed2i" />
@@ -8,11 +21,13 @@
 <xacro:include filename="$(find zed_wrapper)/urdf/zed_macro.urdf.xacro" />
 <!--BASE LINK-->
+<!-- base_link is at wheel axle height (wheel_radius above ground) -->
 <link name = "base_link">
 </link>
 <!--BASEFOOTPRINT LINK-->
+<!-- base_footprint is the ground projection of the robot (at Z=0) -->
 <joint name="basefootprint_joint" type="fixed">
     <parent link="base_link"/>
     <child link="base_footprint"/>
-    <origin xyz="0 0 0" rpy = "0 0 0"/>
+    <origin xyz="0 0 ${-wheel_radius}" rpy = "0 0 0"/>
 </joint>
 <link name="base_footprint">
@@ -28,5 +43,5 @@
         <origin xyz = "0.15 0 0.11" />
         <geometry>
-            <box size = "0.3 0.35 0.22"/>
+            <box size = "${body_length} ${body_width} ${body_height}"/>
         </geometry>
         <material name = "blue">
@@ -37,5 +52,5 @@
         <origin xyz = "0.15 0 0.11" />
        <geometry>
-            <box size = "0.3 0.35 0.22"/>
+            <box size = "${body_length} ${body_width} ${body_height}"/>
         </geometry>
     </collision>
@@ -46,8 +61,9 @@
 </link>
 <!--LEFT WHEEL-->
+<!-- Wheels are at base_link height (Z=0), which is the axle height -->
 <joint name = "left_wheel_joint" type = "continuous">
     <parent link= "base_link"/>
     <child link= "left_wheel_link"/>
-    <origin xyz = "0 0.2 0.05" rpy = "-1.571 3.142 0"/>
+    <origin xyz = "0 ${wheel_base/2} 0" rpy = "-1.571 3.142 0"/>
     <axis xyz = "0 0 1"/>
 </joint>
@@ -55,5 +71,5 @@
     <visual>
         <geometry>
-            <cylinder length = "0.057" radius = "0.08"/>
+            <cylinder length = "${wheel_width}" radius = "${wheel_radius}"/>
         </geometry>
         <material name = "black">
@@ -63,5 +79,5 @@
     <collision>
         <geometry>
-            <cylinder length = "0.057" radius = "0.08"/>
+            <cylinder length = "${wheel_width}" radius = "${wheel_radius}"/>
         </geometry>
     </collision>
@@ -75,5 +91,5 @@
     <parent link = "base_link"/>
     <child link = "right_wheel_link"/>
-    <origin xyz = "0 -0.2 0.05" rpy = "1.571 0 0 "/>
+    <origin xyz = "0 ${-wheel_base/2} 0" rpy = "1.571 0 0 "/>
     <axis xyz = "0 0 -1"/>
 </joint>
@@ -81,5 +97,5 @@
     <visual>
         <geometry>
-            <cylinder length = "0.057" radius = "0.08"/>
+            <cylinder length = "${wheel_width}" radius = "${wheel_radius}"/>
         </geometry>
         <material name = "black">
@@ -89,5 +105,5 @@
     <collision>
         <geometry>
-            <cylinder length = "0.057" radius = "0.08"/>
+            <cylinder length = "${wheel_width}" radius = "${wheel_radius}"/>
         </geometry>
     </collision>
@@ -97,9 +113,10 @@
     </inertial>
 </link>
-<!-- FRONT CASTER WHEELL-->
+<!-- FRONT CASTER WHEEL-->
+<!-- Caster bottom should touch ground: Z = -(wheel_radius - caster_radius) -->
 <link name = "front_caster_wheel_link" >
     <visual>
         <geometry>
-            <sphere radius= "0.03"/>
+            <sphere radius= "${caster_radius}"/>
         </geometry>
         <material name = "red" >
@@ -109,5 +126,5 @@
     <collision>
         <geometry>
-            <sphere radius= "0.03"/>
+            <sphere radius= "${caster_radius}"/>
         </geometry>
     </collision>
@@ -116,11 +133,12 @@
     <parent link = "body_link"/>
     <child link = "front_caster_wheel_link"/>
-    <origin xyz = "0.25 0 0" />
+    <origin xyz = "0.25 0 ${-(wheel_radius - caster_radius)}" />
 </joint>
 <!-- REAR CASTER WHEEL-->
+<!-- Caster bottom should touch ground: Z = -(wheel_radius - caster_radius) -->
 <link name = "rear_caster_wheel_link" >
     <visual>
         <geometry>
-            <sphere radius= "0.03"/>
+            <sphere radius= "${caster_radius}"/>
         </geometry>
         <material name = "purple" >
@@ -130,5 +148,5 @@
     <collision>
         <geometry>
-            <sphere radius= "0.03"/>
+            <sphere radius= "${caster_radius}"/>
         </geometry>
     </collision>
@@ -137,5 +155,5 @@
     <parent link = "body_link"/>
     <child link = "rear_caster_wheel_link"/>
-    <origin xyz = "0.05 0 0" />
+    <origin xyz = "0.05 0 ${-(wheel_radius - caster_radius)}" />
 </joint>
     <!-- LiDAR componenets-->

Commit message: hardware swap: Oradar MS200 → RPLIDAR S2, Wheeltec N100 → HWT901B via WITMotion
- Replaced oradar_lidar driver with rplidar_ros (apt package)
- Replaced wheeltec_n100_imu driver with witmotion_ros2 (patched for Boost.ASIO)
- Added smart device detection with protocol probing for RPLIDAR, BNO055, HWT901B
- Updated URDF: lidar at +7cm from base_link, rpy=(3.14 0 3.14) for RPLIDAR S2
- Fixed scan orientation: clockwise scan, 180° beam filter zone
- Fixed Nav2 global costmap for odom-only mode (rolling window, no static_layer)
- Fixed motor polarity and odometry direction
- Fixed joystick axis mapping for Xbox 360 controller with xpad driver
- Added udev rules for new FTDI/CH340/CP2102 device layout
- Cleaned up old packages: oradar_lidar, ros2_wheeltec_n100_imu, bno055

File: src/shbat_pkg/urdf/sahabat_robot.urdf.xacro (robot description, xacro)
@@ -161,5 +161,5 @@
     <parent link="body_link"/>
     <child link="lidar_link"/>
-    <origin xyz="0.15 0 0.25" rpy="0 0 0"/>
+    <origin xyz="0.22 0 0.25" rpy="3.14 0 3.14"/>
 </joint>
 <link name="lidar_link">
