Commit message: feat: browser operator console and AprilTag/lidar startup localization
Checkpoint of the current workspace. None of the localization changes
have run on the robot yet; the web console was only tested against a
simulated robot in an isolated ROS domain.

Browser operator console (web_console):
- Stdlib HTTP server node: SSE state stream, map PNG, JSON commands
  through the existing /operator services and control lease.
- Web UI (src/shbat_pkg/web): map with lidar/plan/waypoints/routes/
  dock/tags, pose estimate and nav goal tools, waypoint editing and
  patrol, joystick/WASD teleop, AprilTag capture, map loading, E-stop,
  free view rotation dial with soft detents.
- ZED camera MJPEG view with frame-matched AprilTag outlines, encoded
  only while a browser is watching (up to 15 fps, per-viewer cap).
- live_waypoint_editor starts it by default (--no-web, --web-port,
  --no-rviz); a web console failure does not stop the robot stack.

AprilTag + lidar startup localization (from the previous session):
- scan_matcher / scan_localization: correlative lidar-to-map matcher.
- apriltag_landmark_manager: family normalization, distance gate,
  lidar-validated tag poses, realistic AMCL covariance.
- dock_pose_initializer: waits for AMCL, prefers tags, lidar-searches
  around the dock pose, latched /localization/startup_status.
- ZED HD720 with NITROS disabled for apriltag_ros; camera test launch
  and viewer; AprilTag landmark interfaces and RViz panel.

Also includes pending config, launch, map, waypoint and docs changes
already present in the working tree.

Co-Authored-By: Claude Opus 5.5 <noreply@anthropic.com>

File: src/shbat_pkg/urdf/sahabat_robot.urdf.xacro (robot description, xacro)
@@ -24,4 +24,12 @@
 <link name = "base_link">
 </link>
+<!-- IMU LINK -->
+<!-- The IMU driver publishes in imu_link; keep its aligned sensor frame in TF. -->
+<joint name="imu_joint" type="fixed">
+    <parent link="base_link"/>
+    <child link="imu_link"/>
+    <origin xyz="0 0 0" rpy="0 0 0"/>
+</joint>
+<link name="imu_link"/>
 <!--BASEFOOTPRINT LINK-->
 <!-- base_footprint is the ground projection of the robot (at Z=0) -->
